File: Hardware/InkTime_Schematic.sch (EAGLE design)
At the start: 104 parts, among them IC1 BQ25180YBGR_BQ25180YBGR, IC2 RT6160AWSC_RT6160AWSC, IC3 BMA423_BMA423, IC4 DRV2605YZFR_DRV2605YZFR, J1 TC2030-IDC_TC2030-IDC, J2 503480-2400_503480-2400, J3 KH-TYPE-C-16P_KH-TYPE-C-16P, Q1 20V/4.2A/52mΩ/1.4W, Q2 ESP32_C6_LIBRARY_6_SI1308EDL-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, SW1 2025-10-22_07-23-44_LIBRARY_E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, SW2 2025-10-22_07-23-44_LIBRARY_E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, SW3 2025-10-22_07-23-44_LIBRARY_E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, U1 ESP32_C6_LIBRARY_MAX17048G+T10, X1 32MHz, X2 32.768kHz

Commit message: Finished the schematic and the PCB
Parts:
- removed C26: 12pF, InkTime_v5:GRM011R60J152KE01L_2_GRM011R60J152KE01L
- removed C28: 1pF, InkTime_v5:GRM011R60J152KE01L_2_GRM011R60J152KE01L
- removed C35, C36: 1uF, InkTime_v5:PERFECT_0402_CAP_0402
- removed D1: ESP32_C6_LIBRARY_3_USBLC6-2SC6Y, InkTime_v5:ESP32_C6_LIBRARY_3_USBLC6-2SC6Y
- removed IC4: DRV2605YZFR_DRV2605YZFR, InkTime_v5:DRV2605YZFR_DRV2605YZFR
- removed R1, R11: 10K, InkTime_v5:CPF0201D7K68C1_CPF0201D7K68C1
- removed R6: 0, InkTime_v5:CPF0201D7K68C1_CPF0201D7K68C1
- removed U$1: NORDIC_NRF_4_NRF52840_QF, InkTime_v5:NORDIC_NRF_4_NRF52840_QF
- removed U$3: 3.9nH, InkTime_v5:NORDIC_NRF_2_INDUCTOR_0201_L
- added C42: 0.1uF, InkTime_v5:GRM011R60J152KE01L_2_GRM011R60J152KE01L
- added C43: 4.7uF, InkTime_v5:PERFECT_0402_CAP_0402
- added D5: MBR0530, InkTime_v5:ESP32_C6_LIBRARY_5_MBR0530
- added EPD_C1, EPD_C2: 1uF/50V, InkTime_v5:PERFECT_0402_CAP_0402
- added IC9: RT6160AWSC, InkTime_v5:RT6160AWSC_RT6160AWSC
- added L5: 68uH, InkTime_v5:ESP32_C6_LIBRARY_2_744043680IND_4828-WE-TPC_WRE
- added R17, R18: 3K3, InkTime_v5:CPF0201D7K68C1_CPF0201D7K68C1
- added R_TYPE_SEL: 2.2, InkTime_v5:CPF0201D7K68C1_CPF0201D7K68C1
- added TP_VBAT: HECTOR_WATCH_1_TPTP20R, InkTime_v5:HECTOR_WATCH_1_TPTP20R
- added U3: MAX17048G+T10, InkTime_v5:ESP32_C6_LIBRARY_MAX17048G+T10
- ANT1: value 2450AT18B100E_2450AT18B100E -> 2450AT18B100E
- C1: value 1uF -> 12pF; device InkTime_v5:PERFECT_0402_CAP_0402 -> InkTime_v5:GRM011R60J152KE01L_2_GRM011R60J152KE01L
- C10: value 4.7uF -> N.C.; device InkTime_v5:PERFECT_0402_CAP_0402 -> InkTime_v5:GRM011R60J152KE01L_2_GRM011R60J152KE01L
- C11: value 4.7uF -> 100pF; device InkTime_v5:PERFECT_0402_CAP_0402 -> InkTime_v5:GRM011R60J152KE01L_2_GRM011R60J152KE01L
- C12: value 4.7uF -> 100nF; device InkTime_v5:PERFECT_0402_CAP_0402 -> InkTime_v5:GRM011R60J152KE01L_2_GRM011R60J152KE01L
- C13: value 100nF -> N.C.
- C15: value 12pF -> 1.0uF; device InkTime_v5:GRM011R60J152KE01L_2_GRM011R60J152KE01L -> InkTime_v5:PERFECT_0402_CAP_0402
- C16: value 12pF -> 47nF
- C17: value N.C. -> 12pF
- C18: value 100nF -> 12pF
- C19: value 47nF -> 100nF
- C2: value 10uF -> 12pF; device InkTime_v5:PERFECT_0402_CAP_0402 -> InkTime_v5:GRM011R60J152KE01L_2_GRM011R60J152KE01L
- C2-EP-DR: value C2-EP-DR -> 4.7uF/25V
- C20: value 1.0uF -> 4.7uF
- C21: value 100nF -> 4.7uF; device InkTime_v5:GRM011R60J152KE01L_2_GRM011R60J152KE01L -> InkTime_v5:PERFECT_0402_CAP_0402
- C22: value 820pF -> 1pF
- C23: value N.C. -> 0.1uF
- C24: value 100pF -> 10uF; device InkTime_v5:GRM011R60J152KE01L_2_GRM011R60J152KE01L -> InkTime_v5:PERFECT_0402_CAP_0402
- C25: value 12pF -> 22uF; device InkTime_v5:GRM011R60J152KE01L_2_GRM011R60J152KE01L -> InkTime_v5:PERFECT_0402_CAP_0402
- C27: value 1pF -> 0.1uF
- C29: value 1pF -> 1uF; device InkTime_v5:GRM011R60J152KE01L_2_GRM011R60J152KE01L -> InkTime_v5:PERFECT_0402_CAP_0402
- C3: value 1uF -> 1pF; device InkTime_v5:PERFECT_0402_CAP_0402 -> InkTime_v5:GRM011R60J152KE01L_2_GRM011R60J152KE01L
- C30, C38: value 0.1uF -> 1uF; device InkTime_v5:GRM011R60J152KE01L_2_GRM011R60J152KE01L -> InkTime_v5:PERFECT_0402_CAP_0402
- C31: value 4.7uF -> 1uF
- C32: value 1uF/50V -> 1uF
- C33: value 1uF/50V -> 22uF
- C39: value 1uF -> 10uF
- C4: value 22uF -> 1pF; device InkTime_v5:PERFECT_0402_CAP_0402 -> InkTime_v5:GRM011R60J152KE01L_2_GRM011R60J152KE01L
- C5: value 22uF -> 100nF; device InkTime_v5:PERFECT_0402_CAP_0402 -> InkTime_v5:GRM011R60J152KE01L_2_GRM011R60J152KE01L
- C6: value 0.1uF -> 4.7uF; device InkTime_v5:GRM011R60J152KE01L_2_GRM011R60J152KE01L -> InkTime_v5:PERFECT_0402_CAP_0402
- C7: value 10uF -> 100nF; device InkTime_v5:PERFECT_0402_CAP_0402 -> InkTime_v5:GRM011R60J152KE01L_2_GRM011R60J152KE01L
- C9: value 100nF -> 820pF
- D2, D4: value ESP32_C6_LIBRARY_5_MBR0530 -> MBR0530
- D3: value ESP32_C6_LIBRARY_5_MBR0530 -> USBLC6-2SC6Y; device InkTime_v5:ESP32_C6_LIBRARY_5_MBR0530 -> InkTime_v5:ESP32_C6_LIBRARY_3_USBLC6-2SC6Y
- EPD_C5: value 0.1uF -> 0.1uF/50V
- IC1: value BQ25180YBGR_BQ25180YBGR -> BQ25180YBGR
- IC2: value RT6160AWSC_RT6160AWSC -> DRV2605YZFR; device InkTime_v5:RT6160AWSC_RT6160AWSC -> InkTime_v5:DRV2605YZFR_DRV2605YZFR
- J1: value TC2030-IDC_TC2030-IDC -> 503480-2400; device InkTime_v5:TC2030-IDC_TC2030-IDC -> InkTime_v5:503480-2400_503480-2400
- J2: value 503480-2400_503480-2400 -> TC2030-IDC; device InkTime_v5:503480-2400_503480-2400 -> InkTime_v5:TC2030-IDC_TC2030-IDC
- J4: value KH-TYPE-C-16P_KH-TYPE-C-16P -> KH-TYPE-C-16P
- L1: value 68uH -> 3.9nH; device InkTime_v5:ESP32_C6_LIBRARY_2_744043680IND_4828-WE-TPC_WRE -> InkTime_v5:NORDIC_NRF_2_INDUCTOR_0201_L
- L7: value MLP2016SR47MT0S1_FTC252012SR47MBCA -> FTC252012SR47MBCA
- Q1: value 20V/4.2A/52mΩ/1.4W -> DMG2305UX-7 20V/4.2A/52mΩ/1.4W
- Q3: value ESP32_C6_LIBRARY_6_SI1308EDL-T1-GE3 -> SI1308EDL-T1-GE3
- R4: value 3K3 -> 0
- R5: value 3K3 -> 10K
- R7: value 2.2 -> 10K
- U1: value ESP32_C6_LIBRARY_MAX17048G+T10 -> NRF52840_QF; device InkTime_v5:ESP32_C6_LIBRARY_MAX17048G+T10 -> InkTime_v5:NORDIC_NRF_4_NRF52840_QF
- renumbered C40 to C2-EP-DR, C41 to C1_EP-DR, J3 to J4, Q2 to Q3, R10 to R8, SW1 to SW_UP, SW2 to SW_ENT, SW3 to SW_DN
Connections:
- net 3V3: now also C12.2, C19.2, C25.1, C33.1, C34.2, C6.1, C7.2, IC2.VDD, IC9.VOUT_1, IC9.VOUT_2, J2.1, R17.1, R18.1, R5.2, R7.2, U1.VDD@A22, U1.VDD@AD14, U1.VDD@AD23, U1.VDD@B1, U1.VDD@W1, U1.VDDH@Y2; no longer C12.1, C18.2, C21.2, C38.2, C4.1, C5.1, C9.2, IC2.VOUT_1, IC2.VOUT_2, IC4.VDD, J1.1, R11.2, R4.1, R5.1, R9.2, U$1.VDD@A22, U$1.VDD@AD14, U$1.VDD@AD23, U$1.VDD@B1, U$1.VDD@W1, U$1.VDDH@Y2
- net ALERT: now also U1.P0.10/NFC2@J24, U3.!ALERT; no longer U$1.P0.10/NFC2@J24, U1.!ALERT
- net D+: now also D3.I/O2_2, U1.D+@AD6; no longer D1.I/O2_2, U$1.D+@AD6
- net D-: now also D3.I/O1_2, U1.D-@AD4; no longer D1.I/O1_2, U$1.D-@AD4
- net DN: now also D3.I/O1_1; no longer D1.I/O1_1
- net DP: now also D3.I/O2_1; no longer D1.I/O2_1
- net EPD_3V3: now also J1.15, J1.16, L5.2; no longer J2.15, J2.16, L1.2
- net EPD_BUSY: now also J1.9, U1.P0.17@AD12; no longer J2.9, U$1.P0.17@AD12
- net EPD_CS: now also J1.12, U1.P0.05/AIN3@K2; no longer J2.12, U$1.P0.05/AIN3@K2
- net EPD_DC: now also J1.11, U1.P0.15@AD10; no longer J2.11, U$1.P0.15@AD10
- net EPD_RST: now also J1.10, U1.P0.16@AC11; no longer J2.10, U$1.P0.16@AC11
- net GDR: now also J1.2; no longer J2.2
- net GND: now also C10.1, C11.1, C12.1, C19.1, C20.2, C21.2, C23.2, C29.2, C3.1, C30.2, C32.2, C33.2, C38.2, C4.1, C42.1, C43.2, C5.1, D3.GND, EPD_C1.1, EPD_C2.1, IC2.GND, IC2.IN/TRIG, IC9.AGND, IC9.PGND_1, IC9.PGND_2, IC9.VSEL, J1.17, J1.8, J1.MP1, J1.MP2, J2.3, J2.5, R3.2, R9.2, R_TYPE_SEL.1, U1.VSS_PA@F23, U1.VSS_PAD, U3.CTG, U3.EP, U3.GND, U3.QSTRT; no longer C10.2, C11.2, C12.2, C15.1, C16.1, C21.1, C23.1, C26.2, C28.1, C29.1, C3.2, C30.1, C32.1, C33.1, C35.2, C36.2, C38.1, C4.2, C5.2, D1.GND, IC2.AGND, IC2.PGND_1, IC2.PGND_2, IC2.VSEL, IC4.GND, IC4.IN/TRIG, J1.3, J1.5, J2.17, J2.8, J2.MP1, J2.MP2, R1.2, R6.2, R7.1, U$1.VSS_PA@F23, U$1.VSS_PAD, U1.CTG, U1.EP, U1.GND, U1.QSTRT
- net HAPTIC_EN: now also IC2.EN, U1.P0.12@U1; no longer IC4.EN, U$1.P0.12@U1
- net IMU_INT1: now also U1.P0.08@N1; no longer U$1.P0.08@N1
- net IMU_INT2: now also U1.P1.08@P2; no longer U$1.P1.08@P2
- net LX1: now also IC9.SW1_1, IC9.SW1_2; no longer IC2.SW1_1, IC2.SW1_2
- net LX2: now also IC9.SW2_1, IC9.SW2_2; no longer IC2.SW2_1, IC2.SW2_2
- net MOSI: now also J1.14, U1.P0.03/AIN1@B13; no longer J2.14, U$1.P0.03/AIN1@B13
- net N$1: now also IC9.SCL, R4.1; no longer IC2.SCL, R2.1
- net N$11: now also C18.2, U1.P0.01/XL2@F2; no longer C16.2, U$1.P0.01/XL2@F2
- net N$12: now also C15.2, C16.1, U1.VSS@B7; no longer C19.1, C20.2, U$1.VSS@B7
- net N$15: now also C11.2, U1.DEC3@D23; no longer C24.2, U$1.DEC3@D23
- net N$16: now also C2.1, U1.XC2@A23; no longer C25.1, U$1.XC2@A23
- net N$17: now also C1.1, U1.XC1@B24; no longer C26.1, U$1.XC1@B24
- net N$19: now also C3.2, L1.1, U1.ANT@H23; no longer C27.2, U$1.ANT@H23, U$3.1
- net N$2: now also IC9.SDA, R2.1; no longer IC2.SDA, R3.1
- net N$20: now also C22.2, C4.2, L1.2; no longer C28.2, C29.2, U$3.2
- net N$22: now also J1.18; no longer J2.18
- net N$23: now also J1.19; no longer J2.19
- net N$24: now also C13.2, U1.DEC2@A18; no longer C17.2, U$1.DEC2@A18
- net N$25: now also C9.2, U1.DEC5@N24; no longer C22.2, U$1.DEC5@N24
- net N$26: now also J1.20; no longer J2.20
- net N$28: now also J1.22; no longer J2.22
- net N$3: now also C20.1, U1.DEC3V3@AC5; no longer C11.1, U$1.DEC3V3@AC5
- net N$30: now also EPD_C2.2, J1.4; no longer C32.2, J2.4
- net N$31: now also EPD_C1.2, J1.5; no longer C33.2, J2.5
- net N$32: now also J1.24; no longer J2.24
- net N$33: now also R_TYPE_SEL.2; no longer R7.2
- net N$34: now also D5.A, L5.1; no longer D2.A, L1.1
- net N$35: now also C10.2, C15.1, C16.2, U1.DEC4@B5, U1.DEC6@E24; no longer C19.2, C20.1, C23.2, U$1.DEC4@B5, U$1.DEC6@E24
- net N$39: now also D2.K; no longer D3.K
- net N$4: now also C5.2, U1.DEC1@C1; no longer C13.2, U$1.DEC1@C1
- net N$43: now also C32.1, IC2.REG; no longer C39.1, IC4.REG
- net N$5: now also R3.1; no longer R6.1
- net N$6: now also R9.1; no longer R1.1
- net N$7: now also C17.2, U1.P0.00/XL1@D2; no longer C15.2, U$1.P0.00/XL1@D2
- net N$9: now also U1.DCC@B3; no longer U$1.DCC@B3
- net OUT+: now also IC2.OUT+; no longer IC4.OUT+
- net OUT-: now also IC2.OUT-; no longer IC4.OUT-
- net P0.04: now also U1.P0.04/AIN2@J1; no longer U$1.P0.04/AIN2@J1
- net P0.09: now also U1.P0.09/NFC1@L24; no longer U$1.P0.09/NFC1@L24
- net P0.13: now also C30.1, R5.1, U1.P0.13@AD8; no longer C35.1, R9.1, U$1.P0.13@AD8
- net P0.14: now also C31.1, U1.P0.14@AC9; no longer C36.1, U$1.P0.14@AC9
- net P0.19: now also U1.P0.19@AC15; no longer U$1.P0.19@AC15
- net P0.20: now also U1.P0.20@AD16; no longer U$1.P0.20@AD16
- net P0.21: now also U1.P0.21@AC17; no longer U$1.P0.21@AC17
- net P0.22: now also U1.P0.22@AD18; no longer U$1.P0.22@AD18
- net P0.23: now also U1.P0.23@AC19; no longer U$1.P0.23@AC19
- net P0.24: now also U1.P0.24@AD20; no longer U$1.P0.24@AD20
- net P0.25: now also U1.P0.25@AC21; no longer U$1.P0.25@AC21
- net P0.26: now also U1.P0.26@G1; no longer U$1.P0.26@G1
- net P0.27: now also U1.P0.27@H2; no longer U$1.P0.27@H2
- net P0.28: now also U1.P0.28/AIN4@B11; no longer U$1.P0.28/AIN4@B11
- net P0.29: now also U1.P0.29/AIN5@A10; no longer U$1.P0.29/AIN5@A10
- net P0.30: now also U1.P0.30/AIN6@B9; no longer U$1.P0.30/AIN6@B9
- net P0.31: now also U1.P0.31/AIN7@A8; no longer U$1.P0.31/AIN7@A8
- net P1.01: now also U1.P1.01@Y23; no longer U$1.P1.01@Y23
- net P1.02: now also C29.1, R7.1, U1.P1.02@W24; no longer C37.1, R11.1, U$1.P1.02@W24
- net P1.03: now also U1.P1.03@V23; no longer U$1.P1.03@V23
- net P1.04: now also U1.P1.04@U24; no longer U$1.P1.04@U24
- net P1.05: now also U1.P1.05@T23; no longer U$1.P1.05@T23
- net P1.06: now also U1.P1.06@R24; no longer U$1.P1.06@R24
- net P1.07: now also U1.P1.07@P23; no longer U$1.P1.07@P23
- net P1.09: now also U1.P1.09@R1; no longer U$1.P1.09@R1
- net P1.10: now also U1.P1.10@A20; no longer U$1.P1.10@A20
- net P1.11: now also U1.P1.11@B19; no longer U$1.P1.11@B19
- net P1.12: now also U1.P1.12@B17; no longer U$1.P1.12@B17
- net P1.13: now also U1.P1.13@A16; no longer U$1.P1.13@A16
- net P1.14: now also U1.P1.14@B15; no longer U$1.P1.14@B15
- net P1.15: now also U1.P1.15@A14; no longer U$1.P1.15@A14
- net PMIC_INT: now also U1.P0.11@T2; no longer U$1.P0.11@T2
- net PREPGH: now also D5.K, J1.21; no longer D2.K, J2.21
- net PREVGL: now also D2.A, J1.23; no longer D3.A, J2.23
- net RESE: now also J1.3; no longer J2.3
- net RESET: now also J2.6, U1.P0.18/RESET@AC13; no longer J1.6, U$1.P0.18/RESET@AC13
- net SCK: now also J1.13, U1.P0.02/AIN0@A12; no longer J2.13, U$1.P0.02/AIN0@A12
- net SCL: now also IC2.SCL, R17.2, U1.P0.07@M2, U3.SCL; no longer IC4.SCL, R2.2, U$1.P0.07@M2, U1.SCL
- net SDA: now also IC2.SDA, R18.2, R2.2, U1.P0.06@L1, U3.SDA; no longer IC4.SDA, R3.2, R5.2, U$1.P0.06@L1, U1.SDA
- net SWDCLK: now also J2.4, U1.SWDCLK@AA24; no longer J1.4, U$1.SWDCLK@AA24
- net SWDIO: now also J2.2, U1.SWDIO@AC24; no longer J1.2, U$1.SWDIO@AC24
- net SWO: now also U1.P1.00@AD22; no longer U$1.P1.00@AD22
- net VBAT: now also C27.2, C37.1, TP_VBAT.TP, U3.CELL, U3.VDD; no longer C3.1, C30.2, U1.CELL, U1.VDD
- net VBUS: now also C21.1, C38.1, C42.2, C43.1, D3.VBUS, U1.VBUS@AD2; no longer C1.1, C10.1, C31.1, C34.2, D1.VBUS, U$1.VBUS@AD2
- net VREG: now also C23.1, C24.2, C39.1, IC9.EN, IC9.VIN_1, IC9.VIN_2; no longer C2.1, C6.1, C7.2, IC2.EN, IC2.VIN_1, IC2.VIN_2
Other:
- note added: "SWD"
- moved on the sheet: C1, C10, C11, C12, C13, C15, C16, C17, C18, C19, C2, C20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
